File: Blueprint/Wled blueprint.kicad_sch (KiCad schematic)
At the start: 12 parts, among them J1 Conn_01x11, SW1 SW_Push, SW10 SW_Push, SW2 SW_Push, SW3 SW_Push, SW4 SW_Push, SW5 SW_Push, SW6 SW_Push, SW7 SW_Push, SW8 SW_Push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

Commit message: finished wiring diagramm
Connections:
- net Lite: now reaches J1.1 (Pin_1)
- net 3v3: now reaches J1.10 (Pin_10)
- net Vin: now reaches J1.11 (Pin_11)
- net Vin: now also U1.12 (3V3)
- net CCS: now reaches J1.2 (Pin_2)
- net D/C: now reaches J1.3 (Pin_3)
- net D/C: now also U1.10 (GPIO9_D9_MISO)
- net RST: now reaches J1.4 (Pin_4)
- net RST: now also U1.29 (GPIO6_MTCK)
- net TCS: now reaches J1.5 (Pin_5)
- net TCS: now also U1.8 (GPIO20_D7_RX)
- net SI: now reaches J1.6 (Pin_6)
- net SI: now also U1.11 (GPIO10_D10_MOSI)
- net SO: now reaches J1.7 (Pin_7)
- net SCK: now reaches J1.8 (Pin_8)
- net SCK: now also U1.9 (GPIO8_D8_SCK)
- net Gnd: now reaches J1.9 (Pin_9)
- net Gnd: now also U1.13 (GND)
- net GND: now reaches SW5.1
- net GND: now also SW1.1, SW10.1, SW2.1, SW3.1, SW4.1, SW6.1, SW7.1, SW8.1, SW9.1, U1.33 (GND)
- net at SW5.2: now also U1.2 (GPIO3_A1_D1)
- net at SW10.2: now also U1.7 (GPIO21_D6_TX)
- net at SW6.2: now also U1.3 (GPIO4_A2_D2)
- net at SW2.2: now also U1.25 (GPIO7_MTDO)
- net at SW3.2: now also U1.24 (GPIO5_MTDI)
- net at SW9.2: now also U1.6 (GPIO7_D5_SCL)
- net at SW7.2: now also U1.4 (GPIO5_A3_D3)
- net at SW4.2: now also U1.1 (GPIO2_A0_D0)
- net at SW1.2: now also U1.28 (GPIO4_MTMS)
- net at U1.5 (GPIO6_D4_SDA): now also SW8.2
- no-connect marks 0 -> 4

Commit message: fixed 3d model
Parts:
- added BT1: Battery_Cell, symbol Device:Battery_Cell
Connections:
- net GND: now also BT1.2 (-)
- net at U1.32 (BAT): now also BT1.1 (+)
Changed lines of the file:
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@@
+	)
+	(junction
+		(at 135.89 147.32)
+		(diameter 0)
+		(color 0 0 0 0)
 	)
 	(junction
@@
 	(wire
 		(pts
+			(xy 130.81 147.32) (xy 135.89 147.32)
+		)
+		(stroke
+			(width 0)
+			(type default)
+		)
+	)
+	(wire
+		(pts
 			(xy 110.49 118.11) (xy 110.49 134.62)
 		)
@@
 	(wire
 		(pts
+			(xy 130.81 144.78) (xy 130.81 147.32)
+		)
+		(stroke
+			(width 0)
+			(type default)
+		)
+	)
+	(wire
+		(pts
 			(xy 113.03 106.68) (xy 101.6 106.68)
 		)
@@
 	(wire
 		(pts
+			(xy 130.81 132.08) (xy 130.81 137.16)
+		)
+		(stroke
+			(width 0)
+			(type default)
+		)
+	)
+	(wire
+		(pts
 			(xy 172.72 95.25) (xy 177.8 95.25)
 		)
@@
 	(wire
 		(pts
-			(xy 135.89 132.08) (xy 135.89 139.7)
+			(xy 135.89 132.08) (xy 135.89 147.32)
 		)
 		(stroke
@@
 	)
 	(symbol
+		(lib_id "Device:Battery_Cell")
+		(at 130.81 142.24 0)
+		(mirror y)
+		(unit 1)
+		(body_style 1)
+		(exclude_from_sim no)
+		(in_bom yes)
+		(on_board yes)
+		(in_pos_files yes)
+		(dnp no)
+		(property "Reference" "BT1"
+			(at 134.62 139.1284 0)
+			(show_name no)
+			(do_not_autoplace no)
+			(effects
+				(font
+					(size 1.27 1.27)
+				)
+				(justify left)
+			)
+		)
+		(property "Value" "Battery_Cell"
+			(at 130.302 142.748 0)
+			(show_name no)
+			(do_not_autoplace no)
+			(effects
+				(font
+					(size 1.27 1.27)
+				)
+				(justify left)
+			)
+		)
+		(property "Footprint" ""
+			(at 130.81 140.716 90)
+			(hide yes)
+			(show_name no)
+			(do_not_autoplace no)
+			(effects
+				(font
+					(size 1.27 1.27)
+				)
+			)
+		)
+		(property "Datasheet" ""
+			(at 130.81 140.716 90)
+			(hide yes)
+			(show_name no)
+			(do_not_autoplace no)
+			(effects
+				(font
+					(size 1.27 1.27)
+				)
+			)
+		)
+		(property "Description" "Single-cell battery"
+			(at 130.81 142.24 0)
+			(hide yes)
+			(show_name no)
+			(do_not_autoplace no)
+			(effects
+				(font
+					(size 1.27 1.27)
+				)
+			)
+		)
+		(property "Sim.Device" "V"
+			(at 130.81 142.24 0)
+			(hide yes)
+			(show_name no)
+			(do_not_autoplace no)
+			(effects
+				(font
+					(size 1.27 1.27)
+				)
+			)
+		)
+		(property "Sim.Type" "DC"
+			(at 130.81 142.24 0)
+			(hide yes)
+			(show_name no)
+			(do_not_autoplace no)
+			(effects
+				(font
+					(size 1.27 1.27)
+				)
+			)
+		)
+		(property "Sim.Pins" "1=+ 2=-"
+			(at 130.81 142.24 0)
+			(hide yes)
+			(show_name no)
+			(do_not_autoplace no)
+			(effects
+				(font
+					(size 1.27 1.27)
+				)
+			)
+		)
+		(pin "1"
+		)
+		(pin "2"
+		)
+		(instances
+			(project "Wled blueprint"
+				(path "/068793c0-39af-4e31-8189-816ccd1b9268"
+					(reference "BT1")
+					(unit 1)
+				)
+			)
+		)
+	)
+	(symbol
 		(lib_id "Switch:SW_Push")
 		(at 77.47 83.82 0)
@@
 	(symbol
 		(lib_id "power:GND")
-		(at 135.89 139.7 0)
+		(at 135.89 147.32 0)
 		(unit 1)
 		(body_style 1)
@@
 		(fields_autoplaced yes)
 		(property "Reference" "#PWR02"
-			(at 135.89 146.05 0)
+			(at 135.89 153.67 0)
 			(hide yes)
 			(show_name no)
@@
 		)
 		(property "Value" "GND"
-			(at 135.89 144.78 0)
+			(at 135.89 152.4 0)
 			(show_name no)
 			(do_not_autoplace no)
@@
 		)
 		(property "Footprint" ""
-			(at 135.89 139.7 0)
+			(at 135.89 147.32 0)
 			(hide yes)
 			(show_name no)
@@
 		)
 		(property "Datasheet" ""
-			(at 135.89 139.7 0)
+			(at 135.89 147.32 0)
 			(hide yes)
 			(show_name no)
@@
 		)
 		(property "Description" "Power symbol creates a global label with name \"GND\" , ground"
-			(at 135.89 139.7 0)
-			(hide yes)
-			(show_name no)
+			(at 135.89 147.32 0)
+			(hide yes)
+			(show_name no)
